File: UV_led_small.kicad_pcb (KiCad board)
At the start: 2 copper layers, 144 x 80 mm, 32 parts

Commit message: Добавил изображения
Routing:
- net (no net): track 898.9 -> 844.6 mm
Other:
- board size 144 x 80 mm -> 137.2 x 71.3 mm
